Commit message: dodanie napędu na 4 koła, ruch kół działa poprawnie, sterowność ppojazdu jest zła

File: description/robot_core.xacro (robot description, xacro)
@@ -160,5 +160,5 @@
     </gazebo>
     <!-- BACK LEFT WHEEL LINK -->
-    <joint name="back_left_wheel_joint" type="fixed">
+    <joint name="back_left_wheel_joint" type="continuous">
         <parent link="base_link"/>
         <child link="back_left_wheel"/>
@@ -185,9 +185,9 @@
         <material>Gazebo/Blue</material>
         <!-- Makes wheel has no friction -->
-        <mu1 value="0.001"/>
-        <mu2 value="0.001"/>
+        <!-- <mu1 value="0.001"/>
+        <mu2 value="0.001"/> -->
     </gazebo>
     <!-- BACK RIGHT WHEEL LINK -->
-    <joint name="back_right_wheel_joint" type="fixed">
+    <joint name="back_right_wheel_joint" type="continuous">
         <parent link="base_link"/>
         <child link="back_right_wheel"/>
@@ -214,6 +214,6 @@
         <material>Gazebo/Blue</material>
         <!-- Makes wheel has no friction -->
-        <mu1 value="0.001"/>
-        <mu2 value="0.001"/>
+        <!-- <mu1 value="0.001"/>
+        <mu2 value="0.001"/> -->
     </gazebo>
 </robot>

File: description/ros2_control.xacro (robot description, xacro)
@@ -21,4 +21,20 @@
             <state_interface name="position" />
         </joint>
+        <joint name="back_left_wheel_joint">
+            <command_interface name="velocity">
+                <param name="min">-10</param>
+                <param name="max">10</param>
+            </command_interface>
+            <state_interface name="position" />
+            <state_interface name="velocity" />
+        </joint>
+        <joint name="back_right_wheel_joint">
+            <command_interface name="velocity">
+                <param name="min">-10</param>
+                <param name="max">10</param>
+            </command_interface>
+            <state_interface name="position" />
+            <state_interface name="velocity" />
+        </joint>
     </ros2_control>
     <gazebo>
