Commit message: Zmiana do wizualizacji robota piper wraz z rurami
Napisałem od zera kod robota, tak żeby odpowiadał projektowi oraz dodałem rurę po której może się poruszać.

W przyszłości dodać więcej rur oraz ogarnąć sterowanie z dwóch do czterech kół.

File: description/gazebo_control.xacro (robot description, xacro)
@@ -3,9 +3,13 @@
     <gazebo>
         <plugin name="diff_drive" filename="libgazebo_ros_diff_drive.so">
-            <!-- Wheel Information -->
-            <left_joint>left_wheel_joint</left_joint>
-            <right_joint>right_wheel_joint</right_joint>
-            <wheel_separation>0.35</wheel_separation>
-            <wheel_diameter>0.1</wheel_diameter>
+            <!-- wheels -->
+            <!-- <num_wheel_pairs>2</num_wheel_pairs> -->
+            <left_joint>front_left_wheel_joint</left_joint>
+            <!-- <left_joint>back_left_wheel_joint</left_joint> -->
+            <right_joint>front_right_wheel_joint</right_joint>
+            <!-- <right_joint>back_right_wheel_joint</right_joint> -->
+            <!-- kinematics -->
+            <wheel_separation>0.14</wheel_separation>
+            <wheel_diameter>0.06</wheel_diameter>
             <!-- Limits -->
             <max_wheel_torque>200</max_wheel_torque>
@@ -14,7 +18,9 @@
             <odometry_frame>odom</odometry_frame>
             <robot_base_frame>base_link</robot_base_frame>
+            <!-- topic & re remappings -->
             <publish_odom>true</publish_odom>
             <publish_odom_tf>true</publish_odom_tf>
             <publish_wheel_tf>true</publish_wheel_tf>
+            <update_rate>100.0</update_rate>
         </plugin>
     </gazebo>

File: description/lidar.xacro (robot description, xacro)
@@ -1,34 +1,29 @@
 <?xml version="1.0"?>
-<robot xmlns:xacro="http://www.ros.org/wiki/xacro" >
-    <joint name="laser_joint" type="fixed">
+<robot xmlns:xacro="http://www.ros.org/wiki/xacro">
+    <!-- Lidar -->
+    <joint name="lidar_joint" type="fixed">
         <parent link="chassis"/>
-        <child link="laser_frame"/>
-        <origin xyz="0.1 0 0.175" rpy="0 0 0"/>
+        <child link="laser_link"/>
+        <origin xyz="0.107 0 0.14" rpy="0 -${pi/2} -${pi}"/>
     </joint>
-    <link name="laser_frame">
+    <link name="laser_link">
         <visual>
+            <origin xyz="0 0 0.01" rpy="0 0 0"/>
             <geometry>
-                <cylinder radius="0.05" length="0.04"/>
+                <cylinder radius="0.03" length="0.02"/>
             </geometry>
-            <material name="red"/>
-        </visual>
-        <visual>
-            <origin xyz="0 0 -0.05"/>
-            <geometry>
-                <cylinder radius="0.01" length="0.1"/>
-            </geometry>
-            <material name="black"/>
+            <material name="orange red"/>
         </visual>
         <collision>
             <geometry>
-                <cylinder radius="0.05" length="0.04"/>
+                <cylinder radius="0.03" length="0.02"/>
             </geometry>
         </collision>
-        <xacro:inertial_cylinder mass="0.1" length="0.04" radius="0.05">
+        <xacro:inertial_cylinder mass="0.1" length="0.02" radius="0.03">
             <origin xyz="0 0 0" rpy="0 0 0"/>
         </xacro:inertial_cylinder>
     </link>
-    <gazebo reference="laser_frame">
-        <material>Gazebo/Red</material>
+    <gazebo reference="laser_link">
+        <material>Gazebo/RedBright</material>
         <sensor name="laser" type="ray">
             <pose> 0 0 0 0 0 0 </pose>
@@ -44,5 +39,5 @@
                 </scan>
                 <range>
-                    <min>0.15</min>
+                    <min>0.1</min>
                     <max>8</max>
                 </range>

File: description/robot_core.xacro (robot description, xacro)
@@ -1,4 +1,4 @@
 <?xml version="1.0"?>
-<robot xmlns:xacro="http://www.ros.org/wiki/xacro">
+<robot xmlns:xacro="http://www.ros.org/wiki/xacro" >
     <xacro:include filename="inertial_macros.xacro"/>
     <material name="white">
@@ -17,4 +17,10 @@
         <color rgba="1 0 0 1"/>
     </material>
+    <material name="golden rod">
+        <color rgba="0.85 0.64 0.13 1"/>
+    </material>
+    <material name="orange red">
+        <color rgba="1 0.27 0 1"/>
+    </material>
     <!-- BASE LINK -->
     <link name="base_link">
@@ -24,105 +30,190 @@
         <parent link="base_link"/>
         <child link="chassis"/>
-        <origin xyz="-0.1 0 0"/>
+        <origin xyz="0.085 0 0.01"/>
     </joint>
     <link name="chassis">
         <visual>
-            <origin xyz="0.15 0 0.075"/>
-            <geometry>
-                <box size="0.3 0.3 0.15"/>
-            </geometry>
-            <material name="white"/>
-        </visual>
-        <collision>
-            <origin xyz="0.15 0 0.075"/>
-            <geometry>
-                <box size="0.3 0.3 0.15"/>
-            </geometry>
-        </collision>
-        <xacro:inertial_box mass="0.5" x="0.3" y="0.3" z="0.15">
-            <origin xyz="0.15 0 0.075" rpy="0 0 0"/>
+            <origin xyz="0 0 0.02"/>
+            <geometry>
+                <box size="0.17 0.09 0.04"/>
+            </geometry>
+            <material name="orange"/>
+        </visual>
+        <collision>
+            <origin xyz="0 0 0.02"/>
+            <geometry>
+                <box size="0.17 0.09 0.04"/>
+            </geometry>
+        </collision>
+        <xacro:inertial_box mass="1" x="0.17" y="0.09" z="0.04">
+            <origin xyz="0 0 0.02" rpy="0 0 0"/>
         </xacro:inertial_box>
     </link>
     <gazebo reference="chassis">
-        <material>Gazebo/White</material>
-    </gazebo>
-    <!-- LEFT WHEEL LINK -->
-    <joint name="left_wheel_joint" type="continuous">
-        <parent link="base_link"/>
-        <child link="left_wheel"/>
-        <origin xyz="0 0.175 0" rpy="-${pi/2} 0 0"/>
+        <material>Gazebo/Orange</material>
+    </gazebo>
+    <!-- LIDAR HOLDER -->
+    <joint name="lidar_holder_joint" type="fixed">
+        <parent link="chassis"/>
+        <child link="lidar_holder"/>
+        <origin xyz="0.095 0 0.04"/>
+    </joint>
+    <link name="lidar_holder">
+        <visual>
+            <origin xyz="0 0 0.065"/>
+            <geometry>
+                <box size="0.02 0.085 0.13"/>
+            </geometry>
+            <material name="red"/>
+        </visual>
+        <collision>
+            <origin xyz="0 0 0.065"/>
+            <geometry>
+                <box size="0.02 0.085 0.13"/>
+            </geometry>
+        </collision>
+        <xacro:inertial_box mass="0.2" x="0.02" y="0.085" z="0.13">
+            <origin xyz="0 0 0.065" rpy="0 0 0"/>
+        </xacro:inertial_box>
+    </link>
+    <gazebo reference="lidar_holder">
+        <material>Gazebo/Red</material>
+    </gazebo>
+    <!-- UP BOARD -->
+    <joint name="up_board_joint" type="fixed">
+        <parent link="chassis"/>
+        <child link="up_board"/>
+        <origin xyz="-0.05 0 0.04"/>
+    </joint>
+    <link name="up_board">
+        <visual>
+            <origin xyz="0 0 0.02"/>
+            <geometry>
+                <box size="0.056 0.085 0.04"/>
+            </geometry>
+            <material name="golden rod"/>
+        </visual>
+        <collision>
+            <origin xyz="0 0 0.02"/>
+            <geometry>
+                <box size="0.056 0.085 0.04"/>
+            </geometry>
+        </collision>
+        <xacro:inertial_box mass="0.2" x="0.056" y="0.085" z="0.04">
+            <origin xyz="0 0 0.02" rpy="0 0 0"/>
+        </xacro:inertial_box>
+    </link>
+    <gazebo reference="up_board">
+        <material>Gazebo/Gold</material>
+    </gazebo>
+    <!-- FRONT LEFT WHEEL LINK -->
+    <joint name="front_left_wheel_joint" type="continuous">
+        <parent link="base_link"/>
+        <child link="front_left_wheel"/>
+        <origin xyz="0.155 0.07 0.03" rpy="-${pi/2} 0 0" />
         <axis xyz="0 0 1"/>
     </joint>
-    <link name="left_wheel">
-        <visual>
-            <geometry>
-                <cylinder radius="0.05" length="0.04"/>
-            </geometry>
-            <material name="blue"/>
-        </visual>
-        <collision>
-            <geometry>
-                <cylinder radius="0.05" length="0.04"/>
-            </geometry>
-        </collision>
-        <xacro:inertial_cylinder mass="0.1" length="0.04" radius="0.05">
-            <origin xyz="0 0 0" rpy="0 0 0"/>
-        </xacro:inertial_cylinder>
-    </link>
-    <gazebo reference="left_wheel">
-        <material>Gazebo/Blue</material>
-    </gazebo>
-    <!-- RIGHT WHEEL LINK -->
-    <joint name="right_wheel_joint" type="continuous">
-        <parent link="base_link"/>
-        <child link="right_wheel"/>
-        <origin xyz="0 -0.175 0" rpy="${pi/2} 0 0"/>
+    <link name="front_left_wheel">
+        <visual>
+            <geometry>
+                <cylinder radius="0.03" length="0.048"/>
+            </geometry>
+            <material name="blue"/>
+        </visual>
+        <collision>
+            <geometry>
+                <cylinder radius="0.03" length="0.048"/>
+            </geometry>
+        </collision>
+        <xacro:inertial_cylinder mass="0.1" length="0.048" radius="0.03">
+            <origin xyz="0 0 0" rpy="0 0 0"/>
+        </xacro:inertial_cylinder>
+    </link>
+    <gazebo reference="front_left_wheel">
+        <material>Gazebo/Blue</material>
+    </gazebo>
+    <!-- FRONT RIGHT WHEEL LINK -->
+    <joint name="front_right_wheel_joint" type="continuous">
+        <parent link="base_link"/>
+        <child link="front_right_wheel"/>
+        <origin xyz="0.155 -0.07 0.03" rpy="${pi/2} 0 0" />
         <axis xyz="0 0 -1"/>
     </joint>
-    <link name="right_wheel">
-        <visual>
-            <geometry>
-                <cylinder radius="0.05" length="0.04"/>
-            </geometry>
-            <material name="blue"/>
-        </visual>
-        <collision>
-            <geometry>
-                <cylinder radius="0.05" length="0.04"/>
-            </geometry>
-        </collision>
-        <xacro:inertial_cylinder mass="0.1" length="0.04" radius="0.05">
-            <origin xyz="0 0 0" rpy="0 0 0"/>
-        </xacro:inertial_cylinder>
-    </link>
-    <gazebo reference="right_wheel">
-        <material>Gazebo/Blue</material>
-    </gazebo>
-    <!-- CASTER WHEEL LINK -->
-    <joint name="caster_wheel_joint" type="fixed">
-        <parent link="chassis"/>
-        <child link="caster_wheel"/>
-        <origin xyz="0.24 0 0"/>
-    </joint>
-    <link name="caster_wheel">
-        <visual>
-            <geometry>
-                <sphere radius="0.05"/>
-            </geometry>
-            <material name="black"/>
-        </visual>
-        <collision>
-            <geometry>
-                <sphere radius="0.05"/>
-            </geometry>
-        </collision>
-        <xacro:inertial_sphere mass="0.1" radius="0.05">
-            <origin xyz="0 0 0" rpy="0 0 0"/>
-        </xacro:inertial_sphere>
-    </link>
-    <gazebo reference="caster_wheel">
-        <material>Gazebo/Black</material>
+    <link name="front_right_wheel">
+        <visual>
+            <geometry>
+                <cylinder radius="0.03" length="0.048"/>
+            </geometry>
+            <material name="blue"/>
+        </visual>
+        <collision>
+            <geometry>
+                <cylinder radius="0.03" length="0.048"/>
+            </geometry>
+        </collision>
+        <xacro:inertial_cylinder mass="0.1" length="0.048" radius="0.03">
+            <origin xyz="0 0 0" rpy="0 0 0"/>
+        </xacro:inertial_cylinder>
+    </link>
+    <gazebo reference="front_right_wheel">
+        <material>Gazebo/Blue</material>
+    </gazebo>
+    <!-- BACK LEFT WHEEL LINK -->
+    <joint name="back_left_wheel_joint" type="continuous">
+        <parent link="base_link"/>
+        <child link="back_left_wheel"/>
+        <origin xyz="0.015 0.07 0.03" rpy="-${pi/2} 0 0" />
+        <axis xyz="0 0 1"/>
+    </joint>
+    <link name="back_left_wheel">
+        <visual>
+            <geometry>
+                <cylinder radius="0.03" length="0.048"/>
+            </geometry>
+            <material name="blue"/>
+        </visual>
+        <collision>
+            <geometry>
+                <cylinder radius="0.03" length="0.048"/>
+            </geometry>
+        </collision>
+        <xacro:inertial_cylinder mass="0.1" length="0.048" radius="0.03">
+            <origin xyz="0 0 0" rpy="0 0 0"/>
+        </xacro:inertial_cylinder>
+    </link>
+    <gazebo reference="back_left_wheel">
+        <material>Gazebo/Blue</material>
+        <!-- Makes wheel has no friction -->
         <mu1 value="0.001"/>
         <mu2 value="0.001"/>
     </gazebo>
+    <!-- BACK RIGHT WHEEL LINK -->
+    <joint name="back_right_wheel_joint" type="continuous">
+        <parent link="base_link"/>
+        <child link="back_right_wheel"/>
+        <origin xyz="0.015 -0.07 0.03" rpy="${pi/2} 0 0" />
+        <axis xyz="0 0 -1"/>
+    </joint>
+    <link name="back_right_wheel">
+        <visual>
+            <geometry>
+                <cylinder radius="0.03" length="0.048"/>
+            </geometry>
+            <material name="blue"/>
+        </visual>
+        <collision>
+            <geometry>
+                <cylinder radius="0.03" length="0.048"/>
+            </geometry>
+        </collision>
+        <xacro:inertial_cylinder mass="0.1" length="0.048" radius="0.03">
+            <origin xyz="0 0 0" rpy="0 0 0"/>
+        </xacro:inertial_cylinder>
+    </link>
+    <gazebo reference="back_right_wheel">
+        <material>Gazebo/Blue</material>
+        <!-- Makes wheel has no friction -->
+        <mu1 value="0.001"/>
+        <mu2 value="0.001"/>
+    </gazebo>
 </robot>

Commit message: zmiana rozmiaru kół

File: description/gazebo_control.xacro (robot description, xacro)
@@ -11,5 +11,5 @@
             <!-- kinematics -->
             <wheel_separation>0.14</wheel_separation>
-            <wheel_diameter>0.06</wheel_diameter>
+            <wheel_diameter>0.08</wheel_diameter>
             <!-- Limits -->
             <max_wheel_torque>200</max_wheel_torque>

File: description/robot_core.xacro (robot description, xacro)
@@ -109,7 +109,7 @@
     <!-- FRONT LEFT WHEEL LINK -->
     <joint name="front_left_wheel_joint" type="continuous">
-        <parent link="base_link"/>
+        <parent link="chassis"/>
         <child link="front_left_wheel"/>
-        <origin xyz="0.155 0.07 0.03" rpy="-${pi/2} 0 0" />
+        <origin xyz="0.065 0.07 0.02" rpy="-${pi/2} 0 0" />
         <axis xyz="0 0 1"/>
     </joint>
@@ -117,14 +117,14 @@
         <visual>
             <geometry>
-                <cylinder radius="0.03" length="0.048"/>
-            </geometry>
-            <material name="blue"/>
-        </visual>
-        <collision>
-            <geometry>
-                <cylinder radius="0.03" length="0.048"/>
-            </geometry>
-        </collision>
-        <xacro:inertial_cylinder mass="0.1" length="0.048" radius="0.03">
+                <cylinder radius="0.04" length="0.048" n="50"/>
+            </geometry>
+            <material name="blue"/>
+        </visual>
+        <collision>
+            <geometry>
+                <cylinder radius="0.04" length="0.048" n="50"/>
+            </geometry>
+        </collision>
+        <xacro:inertial_cylinder mass="0.1" length="0.048" radius="0.04">
             <origin xyz="0 0 0" rpy="0 0 0"/>
         </xacro:inertial_cylinder>
@@ -135,7 +135,7 @@
     <!-- FRONT RIGHT WHEEL LINK -->
     <joint name="front_right_wheel_joint" type="continuous">
-        <parent link="base_link"/>
+        <parent link="chassis"/>
         <child link="front_right_wheel"/>
-        <origin xyz="0.155 -0.07 0.03" rpy="${pi/2} 0 0" />
+        <origin xyz="0.065 -0.07 0.02" rpy="${pi/2} 0 0" />
         <axis xyz="0 0 -1"/>
     </joint>
@@ -143,14 +143,14 @@
         <visual>
             <geometry>
-                <cylinder radius="0.03" length="0.048"/>
-            </geometry>
-            <material name="blue"/>
-        </visual>
-        <collision>
-            <geometry>
-                <cylinder radius="0.03" length="0.048"/>
-            </geometry>
-        </collision>
-        <xacro:inertial_cylinder mass="0.1" length="0.048" radius="0.03">
+                <cylinder radius="0.04" length="0.048" n="50"/>
+            </geometry>
+            <material name="blue"/>
+        </visual>
+        <collision>
+            <geometry>
+                <cylinder radius="0.04" length="0.048" n="50"/>
+            </geometry>
+        </collision>
+        <xacro:inertial_cylinder mass="0.1" length="0.048" radius="0.04">
             <origin xyz="0 0 0" rpy="0 0 0"/>
         </xacro:inertial_cylinder>
@@ -161,7 +161,7 @@
     <!-- BACK LEFT WHEEL LINK -->
     <joint name="back_left_wheel_joint" type="continuous">
-        <parent link="base_link"/>
+        <parent link="chassis"/>
         <child link="back_left_wheel"/>
-        <origin xyz="0.015 0.07 0.03" rpy="-${pi/2} 0 0" />
+        <origin xyz="-0.07 0.07 0.02" rpy="-${pi/2} 0 0" />
         <axis xyz="0 0 1"/>
     </joint>
@@ -169,14 +169,14 @@
         <visual>
             <geometry>
-                <cylinder radius="0.03" length="0.048"/>
-            </geometry>
-            <material name="blue"/>
-        </visual>
-        <collision>
-            <geometry>
-                <cylinder radius="0.03" length="0.048"/>
-            </geometry>
-        </collision>
-        <xacro:inertial_cylinder mass="0.1" length="0.048" radius="0.03">
+                <cylinder radius="0.04" length="0.048" n="50"/>
+            </geometry>
+            <material name="blue"/>
+        </visual>
+        <collision>
+            <geometry>
+                <cylinder radius="0.04" length="0.048" n="50"/>
+            </geometry>
+        </collision>
+        <xacro:inertial_cylinder mass="0.1" length="0.048" radius="0.04">
             <origin xyz="0 0 0" rpy="0 0 0"/>
         </xacro:inertial_cylinder>
@@ -184,13 +184,10 @@
     <gazebo reference="back_left_wheel">
         <material>Gazebo/Blue</material>
-        <!-- Makes wheel has no friction -->
-        <!-- <mu1 value="0.001"/>
-        <mu2 value="0.001"/> -->
     </gazebo>
     <!-- BACK RIGHT WHEEL LINK -->
     <joint name="back_right_wheel_joint" type="continuous">
-        <parent link="base_link"/>
+        <parent link="chassis"/>
         <child link="back_right_wheel"/>
-        <origin xyz="0.015 -0.07 0.03" rpy="${pi/2} 0 0" />
+        <origin xyz="-0.07 -0.07 0.02" rpy="${pi/2} 0 0" />
         <axis xyz="0 0 -1"/>
     </joint>
@@ -198,14 +195,14 @@
         <visual>
             <geometry>
-                <cylinder radius="0.03" length="0.048"/>
-            </geometry>
-            <material name="blue"/>
-        </visual>
-        <collision>
-            <geometry>
-                <cylinder radius="0.03" length="0.048"/>
-            </geometry>
-        </collision>
-        <xacro:inertial_cylinder mass="0.1" length="0.048" radius="0.03">
+                <cylinder radius="0.04" length="0.048" n="50"/>
+            </geometry>
+            <material name="blue"/>
+        </visual>
+        <collision>
+            <geometry>
+                <cylinder radius="0.04" length="0.048" n="50"/>
+            </geometry>
+        </collision>
+        <xacro:inertial_cylinder mass="0.1" length="0.048" radius="0.04">
             <origin xyz="0 0 0" rpy="0 0 0"/>
         </xacro:inertial_cylinder>
@@ -213,7 +210,4 @@
     <gazebo reference="back_right_wheel">
         <material>Gazebo/Blue</material>
-        <!-- Makes wheel has no friction -->
-        <!-- <mu1 value="0.001"/>
-        <mu2 value="0.001"/> -->
     </gazebo>
 </robot>
