Commit message: integracja ros2_control

File: description/lidar.xacro (robot description, xacro)
@@ -5,5 +5,5 @@
         <parent link="chassis"/>
         <child link="laser_link"/>
-        <origin xyz="0.107 0 0.14" rpy="0 -${pi/2} -${pi}"/>
+        <origin xyz="0.11 0 0.14" rpy="0 -${pi/2} -${pi}"/>
     </joint>
     <link name="laser_link">
@@ -33,7 +33,7 @@
                 <scan>
                     <horizontal>
-                        <samples>360</samples>
-                        <min_angle>-3.14</min_angle>
-                        <max_angle>3.14</max_angle>
+                        <samples>720</samples>
+                        <min_angle>0</min_angle>
+                        <max_angle>6.28</max_angle>
                     </horizontal>
                 </scan>

File: description/robot.urdf.xacro (robot description, xacro)
@@ -2,5 +2,6 @@
 <robot xmlns:xacro="http://www.ros.org/wiki/xacro"  name="piper">
     <xacro:include filename="robot_core.xacro" />
-    <xacro:include filename="gazebo_control.xacro" />
+    <!-- <xacro:include filename="gazebo_control.xacro" /> -->
+    <xacro:include filename="ros2_control.xacro" />
     <xacro:include filename="lidar.xacro" />
 </robot>

File: description/robot_core.xacro (robot description, xacro)
@@ -160,5 +160,5 @@
     </gazebo>
     <!-- BACK LEFT WHEEL LINK -->
-    <joint name="back_left_wheel_joint" type="continuous">
+    <joint name="back_left_wheel_joint" type="fixed">
         <parent link="base_link"/>
         <child link="back_left_wheel"/>
@@ -189,5 +189,5 @@
     </gazebo>
     <!-- BACK RIGHT WHEEL LINK -->
-    <joint name="back_right_wheel_joint" type="continuous">
+    <joint name="back_right_wheel_joint" type="fixed">
         <parent link="base_link"/>
         <child link="back_right_wheel"/>

Commit message: ustawienie lidaru tak jak rzeczywisty

File: description/lidar.xacro (robot description, xacro)
@@ -5,5 +5,5 @@
         <parent link="chassis"/>
         <child link="laser_link"/>
-        <origin xyz="0.11 0 0.14" rpy="0 -${pi/2} -${pi}"/>
+        <origin xyz="0.11 0 0.14" rpy="0 ${pi/2} 0"/>
     </joint>
     <link name="laser_link">
