Commit message: poprawienie położenia sensora imu

File: description/imu.xacro (robot description, xacro)
@@ -5,5 +5,5 @@
         <parent link="chassis"/>
         <child link="imu_link"/>
-        <origin xyz="0 0 0.04"/>
+        <origin xyz="0 0 0.04" rpy="0 0 ${pi/2}"/>
     </joint>
     <link name="imu_link">

Commit message: poprawienie pozycji imu wzgledem fizycznego

File: description/imu.xacro (robot description, xacro)
@@ -5,5 +5,5 @@
         <parent link="chassis"/>
         <child link="imu_link"/>
-        <origin xyz="0 0 0.04" rpy="0 0 ${pi/2}"/>
+        <origin xyz="0 0 0.04" rpy="0 0 -${pi/2}"/>
     </joint>
     <link name="imu_link">
